Commit message: Refactored RL Operational space velocity control

File: yumi_description/urdf/yumi.urdf (robot description, URDF)
Before this commit: robot yumi, 22 links, 21 joints
Links:
- removed link gripper_l_finger_l
- removed link gripper_r_finger_l
- link gripper_l_base: geometry collision mesh filename=package://yumi_description/meshes/gripper/coarse/base.stl; visual mesh filename=package://yumi_description/meshes/gripper/base.stl
- link gripper_l_finger_r: geometry collision mesh filename=package://yumi_description/meshes/gripper/coarse/finger.stl; visual mesh filename=package://yumi_description/meshes/gripper/finger.stl
- link gripper_r_base: geometry collision mesh filename=package://yumi_description/meshes/gripper/coarse/base.stl; visual mesh filename=package://yumi_description/meshes/gripper/base.stl
- link gripper_r_finger_r: geometry collision mesh filename=package://yumi_description/meshes/gripper/coarse/finger.stl; visual mesh filename=package://yumi_description/meshes/gripper/finger.stl
- link yumi_body: geometry collision mesh filename=package://yumi_description/meshes/coarse/body.stl; visual mesh filename=package://yumi_description/meshes/body.stl
- link yumi_link_1_l: geometry collision mesh filename=package://yumi_description/meshes/coarse/link_1.stl; visual mesh filename=package://yumi_description/meshes/link_1.stl
- link yumi_link_1_r: geometry collision mesh filename=package://yumi_description/meshes/coarse/link_1.stl; visual mesh filename=package://yumi_description/meshes/link_1.stl
- link yumi_link_2_l: geometry collision mesh filename=package://yumi_description/meshes/coarse/link_2.stl; visual mesh filename=package://yumi_description/meshes/link_2.stl
- link yumi_link_2_r: geometry collision mesh filename=package://yumi_description/meshes/coarse/link_2.stl; visual mesh filename=package://yumi_description/meshes/link_2.stl
- link yumi_link_3_l: geometry collision mesh filename=package://yumi_description/meshes/coarse/link_3.stl; visual mesh filename=package://yumi_description/meshes/link_3.stl
- link yumi_link_3_r: geometry collision mesh filename=package://yumi_description/meshes/coarse/link_3.stl; visual mesh filename=package://yumi_description/meshes/link_3.stl
- link yumi_link_4_l: geometry collision mesh filename=package://yumi_description/meshes/coarse/link_4.stl; visual mesh filename=package://yumi_description/meshes/link_4.stl
- link yumi_link_4_r: geometry collision mesh filename=package://yumi_description/meshes/coarse/link_4.stl; visual mesh filename=package://yumi_description/meshes/link_4.stl
- link yumi_link_5_l: geometry collision mesh filename=package://yumi_description/meshes/coarse/link_5.stl; visual mesh filename=package://yumi_description/meshes/link_5.stl
- link yumi_link_5_r: geometry collision mesh filename=package://yumi_description/meshes/coarse/link_5.stl; visual mesh filename=package://yumi_description/meshes/link_5.stl
- link yumi_link_6_l: geometry collision mesh filename=package://yumi_description/meshes/coarse/link_6.stl; visual mesh filename=package://yumi_description/meshes/link_6.stl
- link yumi_link_6_r: geometry collision mesh filename=package://yumi_description/meshes/coarse/link_6.stl; visual mesh filename=package://yumi_description/meshes/link_6.stl
- link yumi_link_7_l: geometry collision mesh filename=package://yumi_description/meshes/coarse/link_7.stl; visual mesh filename=package://yumi_description/meshes/link_7.stl
- link yumi_link_7_r: geometry collision mesh filename=package://yumi_description/meshes/coarse/link_7.stl; visual mesh filename=package://yumi_description/meshes/link_7.stl
Joints:
- removed joint gripper_l_joint_m
- removed joint gripper_r_joint_m
- joint gripper_l_joint: type prismatic -> fixed
- joint gripper_r_joint: type prismatic -> fixed

File: yumi_description/urdf/yumi_fixedgrippers.urdf.xacro (robot description, xacro)
@@ -25,3 +25,8 @@
     <origin xyz="0 0 0.007" rpy="0 0 ${PI}" />
   </xacro:yumi_servo_gripper>
+  <gazebo>
+    <plugin name="gazebo_ros_controller" filename="libgazebo_ros_control.so">
+      <robotNamespace>/yumi</robotNamespace>
+    </plugin>
+  </gazebo>
 </robot>

File: yumi_description/urdf/yumi_nogrippers.urdf.xacro (robot description, xacro)
@@ -15,3 +15,8 @@
     <origin xyz="0 0 0.1" rpy="0 0 0" />
   </xacro:yumi>
+  <gazebo>
+    <plugin name="gazebo_ros_controller" filename="libgazebo_ros_control.so">
+      <robotNamespace>/yumi</robotNamespace>
+    </plugin>
+  </gazebo>
 </robot>
