Commit message: Code for Senior design project

File: yumi_description/urdf/yumi_servo_gripper_fixed.xacro (robot description, xacro)
@@ -58,4 +58,6 @@
         <origin xyz="0 0 0" rpy="0 0 0"/>
         <mass value="0.01"/>
+<!-- <mass value="0.01"/> -->
+<mass value="5"/>
         <inertia ixx="0.000001"  ixy="0"  ixz="0" iyy="0.000001" iyz="0" izz="0.000001" />
       </inertial>

File: yumi_description/urdf/yumi_servo_gripper_fixed1.xacro (robot description, xacro)
@@ -22,5 +22,5 @@
       <inertial>
         <origin xyz="0 0 0" rpy="0 0 0"/>
-        <mass value="0.2"/>
+        <mass value="10"/> <!-- 0.2-->
         <inertia ixx="0.0001"  ixy="0"  ixz="0" iyy="0.0001" iyz="0" izz="0.0001" />
       </inertial>
@@ -57,5 +57,5 @@
       <inertial>
         <origin xyz="0 0 0" rpy="0 0 0"/>
-        <mass value="0.01"/>
+        <mass value="0.01"/> <!-- 0.01-->
         <inertia ixx="0.000001"  ixy="0"  ixz="0" iyy="0.000001" iyz="0" izz="0.000001" />
       </inertial>
