Commit message: added new launch files

File: yumi_description/urdf/yumi.xacro (robot description, xacro)
@@ -58,6 +58,6 @@
       <inertial>
         <origin xyz="0 -0.03 0.12" rpy="0 0 0"/>
-        <mass value="2"/>
-        <inertia ixx="0.1"  ixy="0"  ixz="0" iyy="0.1" iyz="0" izz="0.1" />
+        <mass value="0.96"/>
+        <inertia ixx="0.43"  ixy="-0.32"  ixz="0.11" iyy="0.30" iyz="-0.13" izz="0.65" />
       </inertial>
       <visual>
@@ -93,6 +93,6 @@
       <inertial>
         <origin xyz="0 0 0" rpy="0 0 0"/>
-        <mass value="2"/>
-        <inertia ixx="0.1"  ixy="0"  ixz="0" iyy="0.1" iyz="0" izz="0.1" />
+        <mass value="1.41"/>
+        <inertia ixx="0.54"  ixy="-0.45"  ixz="0.09" iyy="0.42" iyz="-0.11" izz="0.91" />
       </inertial>
       <visual>
@@ -128,6 +128,6 @@
       <inertial>
         <origin xyz="0 0 0" rpy="0 0 0"/>
-        <mass value="2"/>
-        <inertia ixx="0.1"  ixy="0"  ixz="0" iyy="0.1" iyz="0" izz="0.1" />
+        <mass value="0.72"/>
+        <inertia ixx="0.22"  ixy="-0.17"  ixz="0.0" iyy="0.13" iyz="-0.01" izz="0.35" />
       </inertial>
       <visual>
@@ -163,6 +163,6 @@
       <inertial>
         <origin xyz="0 0 0" rpy="0 0 0"/>
-        <mass value="2"/>
-        <inertia ixx="0.1"  ixy="0"  ixz="0" iyy="0.1" iyz="0" izz="0.1" />
+        <mass value="1.18"/>
+        <inertia ixx="0.26"  ixy="-0.23"  ixz="0.02" iyy="0.22" iyz="-0.02" izz="0.47" />
       </inertial>
       <visual>
@@ -198,6 +198,6 @@
       <inertial>
         <origin xyz="0 0 0" rpy="0 0 0"/>
-        <mass value="2"/>
-        <inertia ixx="0.1"  ixy="0"  ixz="0" iyy="0.1" iyz="0" izz="0.1" />
+        <mass value="0.34"/>
+        <inertia ixx="0.05"  ixy="-0.07"  ixz="0.01" iyy="0.10" iyz="-0.01" izz="0.15" />
       </inertial>
       <visual>
@@ -233,6 +233,6 @@
       <inertial>
         <origin xyz="0 0 0" rpy="0 0 0"/>
-        <mass value="2"/>
-        <inertia ixx="0.1"  ixy="0"  ixz="0" iyy="0.1" iyz="0" izz="0.1" />
+        <mass value="0.47"/>
+        <inertia ixx="0.05"  ixy="-0.09"  ixz="0.01" iyy="0.15" iyz="-0.01" izz="0.21" />
       </inertial>
       <visual>
@@ -268,6 +268,6 @@
       <inertial>
         <origin xyz="0 0 0" rpy="0 0 0"/>
-        <mass value="2"/>
-        <inertia ixx="0.1"  ixy="0"  ixz="0" iyy="0.1" iyz="0" izz="0.1" />
+        <mass value="0.04"/>
+        <inertia ixx="0.0"  ixy="-0.01"  ixz="0.0" iyy="0.02" iyz="0.0" izz="0.02" />
       </inertial>
       <visual>

File: yumi_description/urdf/yumi_servo_gripper_fixed1.xacro (robot description, xacro)
@@ -22,6 +22,6 @@
       <inertial>
         <origin xyz="0 0 0" rpy="0 0 0"/>
-        <mass value="0.2"/> <!-- 0.2-->
-        <inertia ixx="0.0001"  ixy="0"  ixz="0" iyy="0.0001" iyz="0" izz="0.0001" />
+        <mass value="0.0"/> <!-- 0.2  .2+.5 is max -->
+        <inertia ixx="0.1"  ixy="0"  ixz="0" iyy="0.1" iyz="0" izz="0.1" /> <!-- inertia ixx="0.0001"  ixy="0"  ixz="0" iyy="0.0001" iyz="0" izz="0.0001"-->
       </inertial>
       <visual>
