Commit message: working position state interfaces

File: yumi_description/urdf/yumi.urdf.xacro (robot description, xacro)
@@ -4,5 +4,5 @@
 <!-- |    EDITING THIS FILE BY HAND IS NOT RECOMMENDED                                 | -->
 <!-- =================================================================================== -->
-<robot name="yumi">
+<robot xmlns:xacro="http://wiki.ros.org/xacro" name="yumi">
   <material name="Black">
     <color rgba="0.0 0.0 0.0 1.0"/>
@@ -396,4 +396,26 @@
     </collision>
   </link>
+  <link name="gripper_r_finger_l">
+    <inertial>
+      <origin rpy="0 0 0" xyz="0 0 0"/>
+      <mass value="0.01"/>
+      <!-- 0.01-->
+      <inertia ixx="0.000001" ixy="0" ixz="0" iyy="0.000001" iyz="0" izz="0.000001"/>
+    </inertial>
+    <visual>
+      <origin rpy="0 0 0" xyz="0 0 0"/>
+      <geometry>
+        <mesh filename="package://yumi_description/meshes/gripper/finger.stl"/>
+      </geometry>
+      <material name="Grey"/>
+    </visual>
+    <collision>
+      <origin rpy="0 0 0" xyz="0 0 0"/>
+      <geometry>
+        <mesh filename="package://yumi_description/meshes/gripper/coarse/finger.stl"/>
+      </geometry>
+      <material name="Grey"/>
+    </collision>
+  </link>
   <link name="gripper_l_base">
     <inertial>
@@ -420,4 +442,25 @@
   </link>
   <link name="gripper_l_finger_r">
+    <inertial>
+      <origin rpy="0 0 0" xyz="0 0 0"/>
+      <mass value="0.01"/>
+      <inertia ixx="0.000001" ixy="0" ixz="0" iyy="0.000001" iyz="0" izz="0.000001"/>
+    </inertial>
+    <visual>
+      <origin rpy="0 0 0" xyz="0 0 0"/>
+      <geometry>
+        <mesh filename="package://yumi_description/meshes/gripper/finger.stl"/>
+      </geometry>
+      <material name="Grey"/>
+    </visual>
+    <collision>
+      <origin rpy="0 0 0" xyz="0 0 0"/>
+      <geometry>
+        <mesh filename="package://yumi_description/meshes/gripper/coarse/finger.stl"/>
+      </geometry>
+      <material name="Grey"/>
+    </collision>
+  </link>
+  <link name="gripper_l_finger_l">
     <inertial>
       <origin rpy="0 0 0" xyz="0 0 0"/>
@@ -564,5 +607,4 @@
   </joint>
   <joint name="yumi_link_7_r_joint" type="fixed">
-<!--    <insert_block name="origin"/>-->
     <parent link="yumi_link_7_r"/>
     <child link="gripper_r_base"/>
@@ -573,9 +615,17 @@
     <origin rpy="0 0 0" xyz="0 -0.0065 0.0837"/>
     <axis xyz="-1 0 0"/>
-    <limit effort="300" lower="0" upper="0.025" velocity="0.02"/>
-    <dynamics damping="0.5"/>
+    <limit lower="0" upper="0.025" effort="20.0" velocity="0.02" />
+    <dynamics damping="0.5"/>
+  </joint>
+  <joint name="gripper_r_joint_m" type="prismatic">
+    <parent link="gripper_r_base"/>
+    <child link="gripper_r_finger_l"/>
+    <origin xyz="0 0.0065 0.0837" rpy="0 0 3.1415"/>
+    <axis xyz="-1 0 0"/>
+    <limit lower="0" upper="0.025" effort="20.0" velocity="0.02" />
+    <dynamics damping="0.5"/>
+    <mimic joint="gripper_r_joint"/>
   </joint>
   <joint name="yumi_link_7_l_joint" type="fixed">
-<!--    <insert_block name="origin"/>-->
     <parent link="yumi_link_7_l"/>
     <child link="gripper_l_base"/>
@@ -589,15 +639,31 @@
     <dynamics damping="0.5"/>
   </joint>
+  <joint name="gripper_l_joint_m" type="prismatic">
+    <parent link="gripper_l_base"/>
+    <child link="gripper_l_finger_l"/>
+    <origin xyz="0 0.0065 0.0837" rpy="0 0 3.1415"/>
+    <axis xyz="-1 0 0"/>
+    <limit lower="0" upper="0.025" effort="20.0" velocity="0.02" />
+    <dynamics damping="0.5"/>
+    <mimic joint="gripper_l_joint"/>
+  </joint>
+  <xacro:arg  name="robot_ip" default=""/>
+  <xacro:arg  name="state_server_port_l" default=""/>
+  <xacro:arg  name="state_server_port_r" default=""/>
+  <xacro:arg  name="motion_server_port_l" default=""/>
+  <xacro:arg  name="motion_server_port_r" default=""/>
+  <xacro:arg  name="egm_port_l" default=""/>
+  <xacro:arg  name="egm_port_r" default=""/>
   <!-- ros2 control tag -->
   <ros2_control name="yumi" type="system">
     <hardware>
       <plugin>yumi_hardware/YumiSystem</plugin>
-      <param name="robot_ip">${robot_ip}</param>
-      <param name="state_server_port_l">${state_server_port_l}</param>
-      <param name="state_server_port_r">${state_server_port_r}</param>
-      <param name="motion_server_port_l">${motion_server_port_l}</param>
-      <param name="motion_server_port_r">${motion_server_port_r}</param>
-      <param name="egm_port_l">${egm_port_l}</param>
-      <param name="egm_port_r">${egm_port_r}</param>
+      <param name="robot_ip">$(arg robot_ip)</param>
+      <param name="state_server_port_l">$(arg state_server_port_l)</param>
+      <param name="state_server_port_r">$(arg state_server_port_r)</param>
+      <param name="motion_server_port_l">$(arg motion_server_port_l)</param>
+      <param name="motion_server_port_r">$(arg motion_server_port_r)</param>
+      <param name="egm_port_l">$(arg egm_port_l)</param>
+      <param name="egm_port_r">$(arg egm_port_r)</param>
     </hardware>
     <joint name="yumi_joint_1_r">
@@ -610,4 +676,5 @@
       </state_interface>
       <state_interface name="velocity"/>
+      <state_interface name="effort"/>
     </joint>
     <joint name="yumi_joint_2_r">
@@ -620,4 +687,5 @@
       </state_interface>
       <state_interface name="velocity"/>
+      <state_interface name="effort"/>
     </joint>
     <joint name="yumi_joint_7_r">
@@ -630,4 +698,5 @@
       </state_interface>
       <state_interface name="velocity"/>
+      <state_interface name="effort"/>
     </joint>
     <joint name="yumi_joint_3_r">
@@ -640,4 +709,5 @@
       </state_interface>
       <state_interface name="velocity"/>
+      <state_interface name="effort"/>
     </joint>
     <joint name="yumi_joint_4_r">
@@ -650,4 +720,5 @@
       </state_interface>
       <state_interface name="velocity"/>
+      <state_interface name="effort"/>
     </joint>
     <joint name="yumi_joint_5_r">
@@ -660,4 +731,5 @@
       </state_interface>
       <state_interface name="velocity"/>
+      <state_interface name="effort"/>
     </joint>
     <joint name="yumi_joint_6_r">
@@ -670,4 +742,5 @@
       </state_interface>
       <state_interface name="velocity"/>
+      <state_interface name="effort"/>
     </joint>
     <joint name="yumi_joint_1_l">
@@ -680,4 +753,5 @@
       </state_interface>
       <state_interface name="velocity"/>
+      <state_interface name="effort"/>
     </joint>
     <joint name="yumi_joint_2_l">
@@ -690,4 +764,5 @@
       </state_interface>
       <state_interface name="velocity"/>
+      <state_interface name="effort"/>
     </joint>
     <joint name="yumi_joint_7_l">
@@ -700,4 +775,5 @@
       </state_interface>
       <state_interface name="velocity"/>
+      <state_interface name="effort"/>
     </joint>
     <joint name="yumi_joint_3_l">
@@ -710,4 +786,5 @@
       </state_interface>
       <state_interface name="velocity"/>
+      <state_interface name="effort"/>
     </joint>
     <joint name="yumi_joint_4_l">
@@ -720,4 +797,5 @@
       </state_interface>
       <state_interface name="velocity"/>
+      <state_interface name="effort"/>
     </joint>
     <joint name="yumi_joint_5_l">
@@ -730,4 +808,5 @@
       </state_interface>
       <state_interface name="velocity"/>
+      <state_interface name="effort"/>
     </joint>
     <joint name="yumi_joint_6_l">
@@ -740,24 +819,35 @@
       </state_interface>
       <state_interface name="velocity"/>
+      <state_interface name="effort"/>
     </joint>
     <joint name="gripper_r_joint">
+      <state_interface name="position">
+        <param name="initial_value">0.0</param>
+      </state_interface>
+      <state_interface name="velocity"/>
+      <state_interface name="effort"/>
       <command_interface name="effort">
         <param name="min">-20.0</param>
         <param name="max">20.0</param>
       </command_interface>
-      <state_interface name="position">
-        <param name="initial_value">0.0</param>
-      </state_interface>
-      <state_interface name="velocity"/>
+<!--      <state_interface name="position">-->
+<!--        <param name="initial_value">0.0</param>-->
+<!--      </state_interface>-->
+<!--      <state_interface name="velocity"/>-->
     </joint>
     <joint name="gripper_l_joint">
+      <state_interface name="position">
+        <param name="initial_value">0.0</param>
+      </state_interface>
+      <state_interface name="velocity"/>
+      <state_interface name="effort"/>
       <command_interface name="effort">
         <param name="min">-20.0</param>
         <param name="max">20.0</param>
       </command_interface>
-      <state_interface name="position">
-        <param name="initial_value">0.0</param>
-      </state_interface>
-      <state_interface name="velocity"/>
+<!--      <state_interface name="position">-->
+<!--        <param name="initial_value">0.0</param>-->
+<!--      </state_interface>-->
+<!--      <state_interface name="velocity"/>-->
     </joint>
   </ros2_control>
